Commit message: add extra joint

File: scara_sam_urdf/urdf/scara_sam.urdf (robot description, URDF)
Before this commit: robot scara_sam, 5 links, 4 joints
Links:
- added link link_4, mass 0.113662822206879
- link link_0: geometry collision mesh filename=package://scara_sam_urdf/meshes/link_0.STL; visual mesh filename=package://scara_sam_urdf/meshes/link_0.STL
- link link_1: geometry collision mesh filename=package://scara_sam_urdf/meshes/link_1.STL; visual mesh filename=package://scara_sam_urdf/meshes/link_1.STL
- link link_2: geometry collision mesh filename=package://scara_sam_urdf/meshes/link_2.STL; visual mesh filename=package://scara_sam_urdf/meshes/link_2.STL
- link link_3: geometry collision mesh filename=package://scara_sam_urdf/meshes/link_3.STL; visual mesh filename=package://scara_sam_urdf/meshes/link_3.STL
Joints:
- added joint joint_4: type continuous, parent link_3, child link_4, origin xyz=0 0 0 rpy=0 0 0, axis 0 0 1
